Commit message: fix: offset and link def

File: my_robot.urdf (robot description, URDF)
Before this commit: robot my_robot, 5 links, 4 joints
Joints:
- removed joint base_to_footprint_joint
- added joint base_joint: type fixed, parent base_footprint, child base_link, origin xyz=0 0 0.1 rpy=0 0 0
- joint base_caster_wheel_joint: origin xyz=0.2 0 -0.025 rpy=0 0 0 -> xyz=0.2 0 -0.05 rpy=0 0 0
