Commit message: gz added inertial and collision

File: my_robot_description/urdf/common_properties.xacro (robot description, xacro)
@@ -7,3 +7,45 @@
         <color rgba="0.5 0.5 0.5 1"/>
     </material>
+    <xacro:macro name="box_inertia" params="m x y z o_xyz o_rpy">
+        <inertial>
+            <mass value="${m}"/>
+            <origin xyz="${o_xyz}" rpy="${o_rpy}"/>
+            <inertia
+                ixx="${(1/12.0) * m * (y*y + z*z)}"
+                ixy="0.0"
+                ixz="0.0"
+                iyy="${(1/12.0) * m * (x*x + z*z)}"
+                iyz="0.0"
+                izz="${(1/12.0) * m * (x*x + y*y)}"
+            />
+        </inertial>
+    </xacro:macro>
+    <xacro:macro name="cylinder_inertia" params="m r l o_xyz o_rpy">
+        <inertial>
+            <mass value="${m}"/>
+            <origin xyz="${o_xyz}" rpy="${o_rpy}"/>
+            <inertia
+                ixx="${(1/12.0) * m * (3*r*r + l*l)}"
+                ixy="0.0"
+                ixz="0.0"
+                iyy="${(1/12.0) * m * (3*r*r + l*l)}"
+                iyz="0.0"
+                izz="${(1/2.0) * m * r*r}"
+            />
+        </inertial>
+    </xacro:macro>
+    <xacro:macro name="sphere_inertia" params="m r o_xyz o_rpy">
+        <inertial>
+            <mass value="${m}"/>
+            <origin xyz="${o_xyz}" rpy="${o_rpy}"/>
+            <inertia
+                ixx="${(2/5.0) * m * r*r}"
+                ixy="0.0"
+                ixz="0.0"
+                iyy="${(2/5.0) * m * r*r}"
+                iyz="0.0"
+                izz="${(2/5.0) * m * r*r}"
+            />
+        </inertial>
+    </xacro:macro>
 </robot>

File: my_robot_description/urdf/mobile_base.xacro (robot description, xacro)
@@ -9,10 +9,18 @@
         <link name="${prefix}_wheel_link">
             <visual>
-                <geometry>
-                    <cylinder radius="${wheel_radius}" length="${wheel_width}" />
-                </geometry>
-                <origin xyz="0 0 0" rpy="${pi /2} 0 0" />
+                    <geometry>
+                        <cylinder radius="${wheel_radius}" length="${wheel_width}" />
+                    </geometry>
+                    <origin xyz="0 0 0" rpy="${pi /2.0} 0 0" />
                 <material name="grey"/>
             </visual>
+            <collision>
+                <geometry>
+                    <sphere radius="${wheel_radius}" />
+                </geometry>
+                <origin xyz="0 0 0" rpy="0 0 0" />
+            </collision>
+            <xacro:cylinder_inertia m ="1.0" r="${wheel_radius}" l="${wheel_width}"
+                                    o_xyz="0 0 0" o_rpy="${pi /2.0} 0 0"/>
         </link>
     </xacro:macro>
@@ -23,7 +31,15 @@
                 <box size="${base_length} ${base_width} ${base_height}" />
             </geometry>
-            <origin xyz="0 0 ${base_height/2}" rpy="0 0 0" />
+            <origin xyz="0 0 ${base_height/2.0}" rpy="0 0 0" />
             <material name="blue"/>
         </visual>
+        <collision>
+            <geometry>
+                <box size="${base_length} ${base_width} ${base_height}" />
+            </geometry>
+            <origin xyz="0 0 ${base_height/2.0}" rpy="0 0 0" />
+        </collision>
+        <xacro:box_inertia m ="5.0" x="${base_length}" y="${base_width}" z="${base_height}"
+                            o_xyz="0 0 ${base_height/2.0}" o_rpy="0 0 0"/>
     </link>
     <xacro:wheel_link prefix="right"/>
@@ -32,9 +48,17 @@
         <visual>
             <geometry>
-                <sphere radius="${wheel_radius/2}" />
+                <sphere radius="${wheel_radius/2.0}" />
             </geometry>
             <origin xyz="0 0 0" rpy="0 0 0" />
             <material name="grey"/>
         </visual>
+        <collision>
+            <geometry>
+                <sphere radius="${wheel_radius/2.0}" />
+            </geometry>
+            <origin xyz="0 0 0" rpy="0 0 0" />
+        </collision>
+        <xacro:sphere_inertia m ="0.5" r="${wheel_radius/2.0}"
+                              o_xyz="0 0 0" o_rpy="0 0 0"/>
     </link>
     <joint name="base_joint" type="fixed">
@@ -46,5 +70,5 @@
         <parent link="base_link"/>
         <child link="right_wheel_link"/>
-        <origin xyz="-${base_length/4} -${(base_width + wheel_width)/2} 0" rpy="0 0 0"/>
+        <origin xyz="-${base_length/4.0} -${(base_width + wheel_width)/2.0} 0" rpy="0 0 0"/>
         <axis xyz="0 1 0"/>
     </joint>
@@ -52,5 +76,5 @@
         <parent link="base_link"/>
         <child link="left_wheel_link"/>
-        <origin xyz="-${base_length/4} ${(base_width + wheel_width)/2} 0" rpy="0 0 0"/>
+        <origin xyz="-${base_length/4.0} ${(base_width + wheel_width)/2.0} 0" rpy="0 0 0"/>
         <axis xyz="0 1 0"/>
     </joint>
@@ -58,5 +82,5 @@
         <parent link="base_link"/>
         <child link="caster_wheel_link"/>
-        <origin xyz="${base_length/3} 0 -${wheel_radius/2}" rpy="0 0 0"/>
+        <origin xyz="${base_length/3.0} 0 -${wheel_radius/2.0}" rpy="0 0 0"/>
     </joint>
 </robot>

File: my_robot_description/urdf/my_robot.urdf.xacro (robot description, xacro)
@@ -3,3 +3,4 @@
     <xacro:include filename="$(find my_robot_description)/urdf/common_properties.xacro" />
     <xacro:include filename="$(find my_robot_description)/urdf/mobile_base.xacro" />
+    <xacro:include filename="$(find my_robot_description)/urdf/mobile_base.gazebo.xacro" />
 </robot>
